Commit message: Add new friction gazebo scenarios.

File: src/simulation/gazebo/world_handler/xacro/fwids_vehicle.xacro (robot description, xacro)
@@ -13,4 +13,6 @@
     <xacro:property name="d_l" value="0.5" />
     <xacro:property name="d_r" value="0.5" />
+    <xacro:arg name="wheel_friction" default="0.8" />
+    <xacro:property name="wheel_friction" value="$(arg wheel_friction)" />
     <!-- # define macros -->
     <!-- ## define material colors for URDF -->
@@ -29,4 +31,7 @@
             <mu1>${mu}</mu1>
             <mu2>${mu}</mu2>
+            <kp>1000000.0</kp>
+            <kd>100.0</kd>
+            <minDepth>0.001</minDepth>
         <xacro:insert_block name="color" />
         </gazebo>
@@ -137,5 +142,5 @@
         <inertia ixx="0.01" iyy="0.01" izz="0.01" ixy="0" ixz="0" iyz="0"/>
 	</xacro:link_generator>
-    <xacro:gazebo_material ref="${name}_wheel_base_link" mu="0.8">
+    <xacro:gazebo_material ref="${name}_wheel_base_link" mu="${wheel_friction}">
 		<material>Gazebo/Black</material>
     </xacro:gazebo_material>
@@ -148,5 +153,5 @@
         <inertia ixx="0.01" iyy="0.01" izz="0.01" ixy="0" ixz="0" iyz="0"/>
 	</xacro:link_generator>
-    <xacro:gazebo_material ref="${name}_wheel_suspension" mu="0.8">
+    <xacro:gazebo_material ref="${name}_wheel_suspension" mu="${wheel_friction}">
 		<material>Gazebo/Red</material>
     </xacro:gazebo_material>
@@ -160,5 +165,5 @@
         <inertia ixx="0.01" iyy="0.01" izz="0.01" ixy="0" ixz="0" iyz="0"/>
 	</xacro:link_generator>
-    <xacro:gazebo_material ref="${name}_wheel_steer" mu="0.8">
+    <xacro:gazebo_material ref="${name}_wheel_steer" mu="${wheel_friction}">
 		<material>Gazebo/GreyTransparent</material>
     </xacro:gazebo_material>
@@ -172,5 +177,5 @@
         <inertia ixx="0.0029167" iyy="0.0029167" izz="0.0056250" ixy="0" ixz="0" iyz="0"/>
 	</xacro:link_generator>
-    <xacro:gazebo_material ref="${name}_wheel_rotor" mu="0.8">
+    <xacro:gazebo_material ref="${name}_wheel_rotor" mu="${wheel_friction}">
 		<material>Gazebo/DarkGrey</material>
     </xacro:gazebo_material>
